File: hardware/pcb/out/plant-room-controller-v2-routed.kicad_pcb (KiCad board)
At the start: 2 copper layers, 190 x 130 mm, 53 parts, among them J1 DHT22-1, J10 VALVE 3, J11 VALVE 4, J12 VALVE 5, J13 VALVE 6, J14 LOAD CELL, J15 RAIN, J16 SPARE IN, J2 DHT22-2, J20 RELAY BOARD 2x10, J21 Q17-Q24 SPARE, J3 FLOAT L, J4 FLOAT H, J5 5V IN, J6 12V IN, J7 PUMP, J8 VALVE 1, J9 VALVE 2, U1A ESP32 socket 1x19, U1B ESP32 socket 1x19, U2 OLED DM0054, U3A 595 IN, U3B 595 CASCADE (NC), U3C 595 OUTPUTS Q0-Q23, U4A HX711 LOGIC, U4B HX711 BRIDGE, U5A RAIN LOGIC, U5B RAIN PLATE

Commit message: Use shift register outputs 1-16 only
The 3x74HC595 chain is still clocked as 24 bits (that is its physical
length), but only Q0-Q15 (relay IN1-IN16) are used: Q16-Q23 are held at
the idle level permanently, the relay chase runs 1-16, and the OLED shows
16 output dots (4px wide, 6px pitch).

PCB: removed the J21 spare header for outputs 17-24; those socket pins on
the module are mechanical only. Re-routed (341 segments, 85 vias), DRC
clean at 0.20 mm.

Co-Authored-By: Claude Opus 5.5 <noreply@anthropic.com>
Parts:
- removed J21: Q17-Q24 SPARE, PlantCtl:PinHeader_1x08_P2.54mm
- U3C: value 595 OUTPUTS Q0-Q23 -> 595 OUTPUTS (1-16 USED)
Connections:
- U3C pad 17: SR_Q16 -> (no net)
- U3C pad 18: SR_Q17 -> (no net)
- U3C pad 19: SR_Q18 -> (no net)
- U3C pad 20: SR_Q19 -> (no net)
- U3C pad 21: SR_Q20 -> (no net)
- U3C pad 22: SR_Q21 -> (no net)
- U3C pad 23: SR_Q22 -> (no net)
- U3C pad 24: SR_Q23 -> (no net)
Routing:
- net SR_Q16: track 56.5 -> 0.00 mm, vias 1 -> 0
- net SR_Q17: track 48.5 -> 0.00 mm, vias 1 -> 0
- net SR_Q18: track 43.5 -> 0.00 mm, vias 1 -> 0
- net SR_Q19: track 37.5 -> 0.00 mm, vias 1 -> 0
- net SR_Q20: track 32.0 -> 0.00 mm, vias 1 -> 0
- net SR_Q21: track 27.0 -> 0.00 mm, vias 1 -> 0
- net SR_Q22: track 22.0 -> 0.00 mm, vias 1 -> 0
- net RLY_IN3: track 120.5 -> 98.5 mm
- net RLY_IN5: track 113.0 -> 93.5 mm, vias 3 -> 1
- net RLY_IN7: track 103.5 -> 86.0 mm, vias 2 -> 1
- net SR_Q23: track 17.0 -> 0.00 mm, vias 1 -> 0
- net RLY_IN8: track 108.5 -> 93.0 mm, vias 2 -> 1
- net RLY_IN4: track 124.5 -> 110.0 mm, vias 3 -> 1
- net RLY_IN2: track 124.0 -> 112.0 mm, vias 4 -> 2
- net RLY_IN6: track 116.5 -> 105.5 mm, vias 3 -> 1
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
Commit message: 17 relay outputs, log each completed relay cycle, MQTT watch tool
- Shift register now drives outputs 1-17: Q0-Q15 to the 16-channel relay
  board (ribbon J20, unchanged), Q16 to a separate single relay on the new
  PCB header J21 (IN/5V/GND). Q17-Q23 stay idle. OLED shows 17 dots
  (5px pitch).
- The relay chase logs one line per completed cycle ("relay chase: cycle
  N complete") to serial and the remote log - batched every 10s, so at
  most one MQTT message per batch.
- tools/mqtt_watch.py: live view of one board's MQTT traffic (logs,
  telemetry, events, config/commands) straight from the broker.
- PCB re-routed (371 segments, 87 vias), DRC clean at 0.20 mm.

Co-Authored-By: Claude Opus 5.5 <noreply@anthropic.com>
Parts:
- added J21: RELAY 17, PlantCtl:PinHeader_1x03_P2.54mm, F.Cu at (137.0, 42.0)
- U3C: value 595 OUTPUTS (1-16 USED) -> 595 OUTPUTS (1-17 USED)
Connections:
- U3C pad 17: (no net) -> RLY_IN17
Routing:
- net RLY_IN17: track 0.00 -> 52.5 mm, vias 0 -> 1
- net GND: track 414.0 -> 443.5 mm, vias 8 -> 9
- net +5V: track 261.0 -> 277.0 mm, vias 3 -> 4
- net RLY_IN11: track 68.0 -> 79.0 mm, vias 2 -> 1
- net RLY_IN3: track 98.5 -> 108.0 mm, vias 3 -> 1
- net RLY_IN1: track 114.0 -> 106.0 mm, vias 2 -> 4
- net RLY_IN4: track 110.0 -> 117.0 mm
- net RLY_IN10: track 79.5 -> 86.5 mm, vias 2 -> 1
- net RLY_IN8: track 93.0 -> 99.0 mm
- net RLY_IN6: track 105.5 -> 111.5 mm, vias 1 -> 2
- net RLY_IN15: track 55.5 -> 52.5 mm, vias 1 -> 0
- net RLY_IN14: track 60.0 -> 62.5 mm
- net RLY_IN5: track 93.5 -> 91.5 mm, vias 1 -> 3
- net RLY_IN2: track 112.0 -> 110.0 mm, vias 2 -> 3
- net RLY_IN12: track 70.0 -> 71.5 mm
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
Commit message: Relay safety at power-up: chase off, outputs latched first, coil power enable
Pumps and valves are now connected, so:
- The relay chase is off by default again (SR_TEST_ENABLED 0).
- setup() latches the all-relays-off frame into the 74HC595s as its very
  first action (it used to run ~3s in, after the splash and a delay).
- New master relay-coil power enable on GPIO2 (LOW through every
  power-up, reset and OTA reboot - the ESP32 itself requires it): it is
  switched on only at the end of setup(), 200ms after the outputs are
  latched off, and switched off again before an OTA download. Drives a
  high-level-trigger single relay module on the new PCB header J22 whose
  NO contact feeds the relay board's JD-VCC, so no relay can energize
  during start-up whatever the shift register outputs do.

PCB: J22 (EN/5V/GND) added, re-routed (387 segments, 90 vias), DRC clean.

Co-Authored-By: Claude Opus 5.5 <noreply@anthropic.com>
Parts:
- added J22: RELAY PWR EN, PlantCtl:PinHeader_1x03_P2.54mm, F.Cu at (137.0, 52.0)
Connections:
- U1B pad 15: (no net) -> RELAY_PWR_EN
Routing:
- net RELAY_PWR_EN: track 0.00 -> 156.0 mm, vias 0 -> 1
- net GND: track 443.5 -> 433.5 mm
- net DHT1_DATA: track 137.5 -> 147.0 mm, vias 3 -> 4
- net RLY_IN2: track 110.0 -> 115.0 mm, vias 3 -> 2
- net RLY_IN10: track 86.5 -> 81.5 mm, vias 1 -> 2
- net RLY_IN11: track 79.0 -> 74.5 mm
- net RLY_IN1: track 106.0 -> 110.0 mm, vias 4 -> 3
- net RLY_IN4: track 117.0 -> 113.5 mm, vias 1 -> 2
- net RLY_IN8: track 99.0 -> 96.0 mm
- net RLY_IN6: track 111.5 -> 108.5 mm
- net RLY_IN12: track 71.5 -> 74.0 mm
- net +5V: track 277.0 -> 279.5 mm
- net RLY_IN3: track 108.0 -> 106.5 mm, vias 1 -> 2
- net RLY_IN5: track 91.5 -> 90.5 mm
