File: hardware/pcb/out/plant-room-controller-v2.kicad_pcb (KiCad board)
At the start: 2 copper layers, 190 x 130 mm, 53 parts, among them J1 DHT22-1, J10 VALVE 3, J11 VALVE 4, J12 VALVE 5, J13 VALVE 6, J14 LOAD CELL, J15 RAIN, J16 SPARE IN, J2 DHT22-2, J20 RELAY BOARD 2x10, J21 Q17-Q24 SPARE, J3 FLOAT L, J4 FLOAT H, J5 5V IN, J6 12V IN, J7 PUMP, J8 VALVE 1, J9 VALVE 2, U1A ESP32 socket 1x19, U1B ESP32 socket 1x19, U2 OLED DM0054, U3A 595 IN, U3B 595 CASCADE (NC), U3C 595 OUTPUTS Q0-Q23, U4A HX711 LOGIC, U4B HX711 BRIDGE, U5A RAIN LOGIC, U5B RAIN PLATE

Commit message: Use shift register outputs 1-16 only
The 3x74HC595 chain is still clocked as 24 bits (that is its physical
length), but only Q0-Q15 (relay IN1-IN16) are used: Q16-Q23 are held at
the idle level permanently, the relay chase runs 1-16, and the OLED shows
16 output dots (4px wide, 6px pitch).

PCB: removed the J21 spare header for outputs 17-24; those socket pins on
the module are mechanical only. Re-routed (341 segments, 85 vias), DRC
clean at 0.20 mm.

Co-Authored-By: Claude Opus 5.5 <noreply@anthropic.com>
Parts:
- removed J21: Q17-Q24 SPARE, PlantCtl:PinHeader_1x08_P2.54mm
- U3C: value 595 OUTPUTS Q0-Q23 -> 595 OUTPUTS (1-16 USED)
Connections:
- U3C pad 17: SR_Q16 -> (no net)
- U3C pad 18: SR_Q17 -> (no net)
- U3C pad 19: SR_Q18 -> (no net)
- U3C pad 20: SR_Q19 -> (no net)
- U3C pad 21: SR_Q20 -> (no net)
- U3C pad 22: SR_Q21 -> (no net)
- U3C pad 23: SR_Q22 -> (no net)
- U3C pad 24: SR_Q23 -> (no net)
Changed lines of the file:
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@@
   (net 55 "RLY_IN15")
   (net 56 "RLY_IN16")
-  (net 57 "SR_Q16")
-  (net 58 "SR_Q17")
-  (net 59 "SR_Q18")
-  (net 60 "SR_Q19")
-  (net 61 "SR_Q20")
-  (net 62 "SR_Q21")
-  (net 63 "SR_Q22")
-  (net 64 "SR_Q23")
   (footprint "PlantCtl:PinSocket_1x19_P2.54mm" (layer "F.Cu")
     (at 17.300 78.780)
@@
     (attr through_hole)
     (fp_text reference "U3C" (at -3.600 0.000) (layer "F.SilkS") (effects (font (size 1 1) (thickness 0.15))))
-    (fp_text value "595 OUTPUTS Q0-Q23" (at 0 -4) (layer "F.Fab") (effects (font (size 1 1) (thickness 0.15))))
+    (fp_text value "595 OUTPUTS (1-16 USED)" (at 0 -4) (layer "F.Fab") (effects (font (size 1 1) (thickness 0.15))))
     (fp_line (start -1.270 -1.270) (end 59.690 -1.270) (layer "F.SilkS") (width 0.12))
     (fp_line (start 59.690 -1.270) (end 59.690 1.270) (layer "F.SilkS") (width 0.12))
@@
     (pad "15" thru_hole circle (at 35.560 0.000) (size 1.7 1.7) (drill 1.0) (layers *.Cu *.Mask) (net 55 "RLY_IN15"))
     (pad "16" thru_hole circle (at 38.100 0.000) (size 1.7 1.7) (drill 1.0) (layers *.Cu *.Mask) (net 56 "RLY_IN16"))
-    (pad "17" thru_hole circle (at 40.640 0.000) (size 1.7 1.7) (drill 1.0) (layers *.Cu *.Mask) (net 57 "SR_Q16"))
-    (pad "18" thru_hole circle (at 43.180 0.000) (size 1.7 1.7) (drill 1.0) (layers *.Cu *.Mask) (net 58 "SR_Q17"))
-    (pad "19" thru_hole circle (at 45.720 0.000) (size 1.7 1.7) (drill 1.0) (layers *.Cu *.Mask) (net 59 "SR_Q18"))
-    (pad "20" thru_hole circle (at 48.260 0.000) (size 1.7 1.7) (drill 1.0) (layers *.Cu *.Mask) (net 60 "SR_Q19"))
-    (pad "21" thru_hole circle (at 50.800 0.000) (size 1.7 1.7) (drill 1.0) (layers *.Cu *.Mask) (net 61 "SR_Q20"))
-    (pad "22" thru_hole circle (at 53.340 0.000) (size 1.7 1.7) (drill 1.0) (layers *.Cu *.Mask) (net 62 "SR_Q21"))
-    (pad "23" thru_hole circle (at 55.880 0.000) (size 1.7 1.7) (drill 1.0) (layers *.Cu *.Mask) (net 63 "SR_Q22"))
-    (pad "24" thru_hole circle (at 58.420 0.000) (size 1.7 1.7) (drill 1.0) (layers *.Cu *.Mask) (net 64 "SR_Q23"))
+    (pad "17" thru_hole circle (at 40.640 0.000) (size 1.7 1.7) (drill 1.0) (layers *.Cu *.Mask))
+    (pad "18" thru_hole circle (at 43.180 0.000) (size 1.7 1.7) (drill 1.0) (layers *.Cu *.Mask))
+    (pad "19" thru_hole circle (at 45.720 0.000) (size 1.7 1.7) (drill 1.0) (layers *.Cu *.Mask))
+    (pad "20" thru_hole circle (at 48.260 0.000) (size 1.7 1.7) (drill 1.0) (layers *.Cu *.Mask))
+    (pad "21" thru_hole circle (at 50.800 0.000) (size 1.7 1.7) (drill 1.0) (layers *.Cu *.Mask))
+    (pad "22" thru_hole circle (at 53.340 0.000) (size 1.7 1.7) (drill 1.0) (layers *.Cu *.Mask))
+    (pad "23" thru_hole circle (at 55.880 0.000) (size 1.7 1.7) (drill 1.0) (layers *.Cu *.Mask))
+    (pad "24" thru_hole circle (at 58.420 0.000) (size 1.7 1.7) (drill 1.0) (layers *.Cu *.Mask))
   )
   (footprint "PlantCtl:IDC_BoxHeader_2x10_P2.54mm" (layer "F.Cu")
@@
     (pad "20" thru_hole circle (at 2.540 22.860) (size 1.7 1.7) (drill 1.0) (layers *.Cu *.Mask) (net 1 "GND"))
   )
-  (footprint "PlantCtl:PinHeader_1x08_P2.54mm" (layer "F.Cu")
-    (at 137.000 42.000)
-    (attr through_hole)
-    (fp_text reference "J21" (at 0.000 -2.400) (layer "F.SilkS") (effects (font (size 1 1) (thickness 0.15))))
-    (fp_text value "Q17-Q24 SPARE" (at 0 -4) (layer "F.Fab") (effects (font (size 1 1) (thickness 0.15))))
-    (fp_line (start -1.270 -1.270) (end 1.270 -1.270) (layer "F.SilkS") (width 0.12))
-    (fp_line (start 1.270 -1.270) (end 1.270 19.050) (layer "F.SilkS") (width 0.12))
-    (fp_line (start 1.270 19.050) (end -1.270 19.050) (layer "F.SilkS") (width 0.12))
-    (fp_line (start -1.270 19.050) (end -1.270 -1.270) (layer "F.SilkS") (width 0.12))
-    (fp_text user "17" (at -2.360 0.000) (layer "F.SilkS") (effects (font (size 0.8 0.8) (thickness 0.12))))
-    (fp_text user "18" (at -2.360 2.540) (layer "F.SilkS") (effects (font (size 0.8 0.8) (thickness 0.12))))
-    (fp_text user "19" (at -2.360 5.080) (layer "F.SilkS") (effects (font (size 0.8 0.8) (thickness 0.12))))
-    (fp_text user "20" (at -2.360 7.620) (layer "F.SilkS") (effects (font (size 0.8 0.8) (thickness 0.12))))
-    (fp_text user "21" (at -2.360 10.160) (layer "F.SilkS") (effects (font (size 0.8 0.8) (thickness 0.12))))
-    (fp_text user "22" (at -2.360 12.700) (layer "F.SilkS") (effects (font (size 0.8 0.8) (thickness 0.12))))
-    (fp_text user "23" (at -2.360 15.240) (layer "F.SilkS") (effects (font (size 0.8 0.8) (thickness 0.12))))
-    (fp_text user "24" (at -2.360 17.780) (layer "F.SilkS") (effects (font (size 0.8 0.8) (thickness 0.12))))
-    (pad "1" thru_hole rect (at 0.000 0.000) (size 1.7 1.7) (drill 1.0) (layers *.Cu *.Mask) (net 57 "SR_Q16"))
-    (pad "2" thru_hole circle (at 0.000 2.540) (size 1.7 1.7) (drill 1.0) (layers *.Cu *.Mask) (net 58 "SR_Q17"))
-    (pad "3" thru_hole circle (at 0.000 5.080) (size 1.7 1.7) (drill 1.0) (layers *.Cu *.Mask) (net 59 "SR_Q18"))
-    (pad "4" thru_hole circle (at 0.000 7.620) (size 1.7 1.7) (drill 1.0) (layers *.Cu *.Mask) (net 60 "SR_Q19"))
-    (pad "5" thru_hole circle (at 0.000 10.160) (size 1.7 1.7) (drill 1.0) (layers *.Cu *.Mask) (net 61 "SR_Q20"))
-    (pad "6" thru_hole circle (at 0.000 12.700) (size 1.7 1.7) (drill 1.0) (layers *.Cu *.Mask) (net 62 "SR_Q21"))
-    (pad "7" thru_hole circle (at 0.000 15.240) (size 1.7 1.7) (drill 1.0) (layers *.Cu *.Mask) (net 63 "SR_Q22"))
-    (pad "8" thru_hole circle (at 0.000 17.780) (size 1.7 1.7) (drill 1.0) (layers *.Cu *.Mask) (net 64 "SR_Q23"))
-  )
   (footprint "PlantCtl:PinSocket_1x04_P2.54mm" (layer "F.Cu")

Commit message: 17 relay outputs, log each completed relay cycle, MQTT watch tool
- Shift register now drives outputs 1-17: Q0-Q15 to the 16-channel relay
  board (ribbon J20, unchanged), Q16 to a separate single relay on the new
  PCB header J21 (IN/5V/GND). Q17-Q23 stay idle. OLED shows 17 dots
  (5px pitch).
- The relay chase logs one line per completed cycle ("relay chase: cycle
  N complete") to serial and the remote log - batched every 10s, so at
  most one MQTT message per batch.
- tools/mqtt_watch.py: live view of one board's MQTT traffic (logs,
  telemetry, events, config/commands) straight from the broker.
- PCB re-routed (371 segments, 87 vias), DRC clean at 0.20 mm.

Co-Authored-By: Claude Opus 5.5 <noreply@anthropic.com>
Parts:
- added J21: RELAY 17, PlantCtl:PinHeader_1x03_P2.54mm, F.Cu at (137.0, 42.0)
- U3C: value 595 OUTPUTS (1-16 USED) -> 595 OUTPUTS (1-17 USED)
Connections:
- U3C pad 17: (no net) -> RLY_IN17
Changed lines of the file:
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@@
   (net 55 "RLY_IN15")
   (net 56 "RLY_IN16")
+  (net 57 "RLY_IN17")
   (footprint "PlantCtl:PinSocket_1x19_P2.54mm" (layer "F.Cu")
     (at 17.300 78.780)
@@
     (attr through_hole)
     (fp_text reference "U3C" (at -3.600 0.000) (layer "F.SilkS") (effects (font (size 1 1) (thickness 0.15))))
-    (fp_text value "595 OUTPUTS (1-16 USED)" (at 0 -4) (layer "F.Fab") (effects (font (size 1 1) (thickness 0.15))))
+    (fp_text value "595 OUTPUTS (1-17 USED)" (at 0 -4) (layer "F.Fab") (effects (font (size 1 1) (thickness 0.15))))
     (fp_line (start -1.270 -1.270) (end 59.690 -1.270) (layer "F.SilkS") (width 0.12))
     (fp_line (start 59.690 -1.270) (end 59.690 1.270) (layer "F.SilkS") (width 0.12))
@@
     (pad "15" thru_hole circle (at 35.560 0.000) (size 1.7 1.7) (drill 1.0) (layers *.Cu *.Mask) (net 55 "RLY_IN15"))
     (pad "16" thru_hole circle (at 38.100 0.000) (size 1.7 1.7) (drill 1.0) (layers *.Cu *.Mask) (net 56 "RLY_IN16"))
-    (pad "17" thru_hole circle (at 40.640 0.000) (size 1.7 1.7) (drill 1.0) (layers *.Cu *.Mask))
+    (pad "17" thru_hole circle (at 40.640 0.000) (size 1.7 1.7) (drill 1.0) (layers *.Cu *.Mask) (net 57 "RLY_IN17"))
     (pad "18" thru_hole circle (at 43.180 0.000) (size 1.7 1.7) (drill 1.0) (layers *.Cu *.Mask))
     (pad "19" thru_hole circle (at 45.720 0.000) (size 1.7 1.7) (drill 1.0) (layers *.Cu *.Mask))
@@
     (pad "20" thru_hole circle (at 2.540 22.860) (size 1.7 1.7) (drill 1.0) (layers *.Cu *.Mask) (net 1 "GND"))
   )
+  (footprint "PlantCtl:PinHeader_1x03_P2.54mm" (layer "F.Cu")
+    (at 137.000 42.000)
+    (attr through_hole)
+    (fp_text reference "J21" (at 0.000 -2.400) (layer "F.SilkS") (effects (font (size 1 1) (thickness 0.15))))
+    (fp_text value "RELAY 17" (at 0 -4) (layer "F.Fab") (effects (font (size 1 1) (thickness 0.15))))
+    (fp_line (start -1.270 -1.270) (end 1.270 -1.270) (layer "F.SilkS") (width 0.12))
+    (fp_line (start 1.270 -1.270) (end 1.270 6.350) (layer "F.SilkS") (width 0.12))
+    (fp_line (start 1.270 6.350) (end -1.270 6.350) (layer "F.SilkS") (width 0.12))
+    (fp_line (start -1.270 6.350) (end -1.270 -1.270) (layer "F.SilkS") (width 0.12))
+    (fp_text user "IN" (at -2.360 0.000) (layer "F.SilkS") (effects (font (size 0.8 0.8) (thickness 0.12))))
+    (fp_text user "5V" (at -2.360 2.540) (layer "F.SilkS") (effects (font (size 0.8 0.8) (thickness 0.12))))
+    (fp_text user "GND" (at -2.690 5.080) (layer "F.SilkS") (effects (font (size 0.8 0.8) (thickness 0.12))))
+    (pad "1" thru_hole rect (at 0.000 0.000) (size 1.7 1.7) (drill 1.0) (layers *.Cu *.Mask) (net 57 "RLY_IN17"))
+    (pad "2" thru_hole circle (at 0.000 2.540) (size 1.7 1.7) (drill 1.0) (layers *.Cu *.Mask) (net 3 "+5V"))
+    (pad "3" thru_hole circle (at 0.000 5.080) (size 1.7 1.7) (drill 1.0) (layers *.Cu *.Mask) (net 1 "GND"))
+  )
   (footprint "PlantCtl:PinSocket_1x04_P2.54mm" (layer "F.Cu")

Commit message: Relay safety at power-up: chase off, outputs latched first, coil power enable
Pumps and valves are now connected, so:
- The relay chase is off by default again (SR_TEST_ENABLED 0).
- setup() latches the all-relays-off frame into the 74HC595s as its very
  first action (it used to run ~3s in, after the splash and a delay).
- New master relay-coil power enable on GPIO2 (LOW through every
  power-up, reset and OTA reboot - the ESP32 itself requires it): it is
  switched on only at the end of setup(), 200ms after the outputs are
  latched off, and switched off again before an OTA download. Drives a
  high-level-trigger single relay module on the new PCB header J22 whose
  NO contact feeds the relay board's JD-VCC, so no relay can energize
  during start-up whatever the shift register outputs do.

PCB: J22 (EN/5V/GND) added, re-routed (387 segments, 90 vias), DRC clean.

Co-Authored-By: Claude Opus 5.5 <noreply@anthropic.com>
Parts:
- added J22: RELAY PWR EN, PlantCtl:PinHeader_1x03_P2.54mm, F.Cu at (137.0, 52.0)
Connections:
- U1B pad 15: (no net) -> RELAY_PWR_EN
